Commit message: feat: Replace empty world with simple-building world

File: my_robot/urdf/my_robot.xacro (robot description, xacro)
@@ -34,28 +34,4 @@
       </geometry>
       <material name="blue"/>
-    </visual>
-    <collision name='back_caster_collision'>
-      <origin xyz="-0.15 0 -0.05" rpy=" 0 0 0"/>
-      <geometry>
-        <sphere radius="0.0499"/>
-      </geometry>
-    </collision>
-    <visual name='back_caster_visual'>
-      <origin xyz="-0.15 0 -0.05" rpy=" 0 0 0"/>
-      <geometry>
-        <sphere radius="0.05"/>
-      </geometry>
-    </visual>
-    <collision name='front_caster_collision'>
-      <origin xyz="0.15 0 -0.05" rpy=" 0 0 0"/>
-      <geometry>
-        <sphere radius="0.0499"/>
-      </geometry>
-    </collision>
-    <visual name='front_caster_visual'>
-      <origin xyz="0.15 0 -0.05" rpy=" 0 0 0"/>
-      <geometry>
-        <sphere radius="0.05"/>
-      </geometry>
     </visual>
   </link>
@@ -170,5 +146,5 @@
     <child link="right_wheel"/>
     <parent link="chassis"/>
-    <axis xyz="0 1 0" rpy="0 0 0"/>
+    <axis xyz="0 -1 0" rpy="0 0 0"/>
     <limit effort="10000" velocity="1000"/>
     <dynamics damping="1.0" friction="1.0"/>

Commit message: fix: Robot wheel collision change to match visual

File: my_robot/urdf/my_robot.xacro (robot description, xacro)
@@ -52,5 +52,5 @@
       />
     </inertial>
-    <collision name='collision'>
+    <collision name='left_collision'>
       <origin xyz="0 0 0" rpy=" 0 1.5707 1.5707"/>
       <geometry>
@@ -75,6 +75,6 @@
       />
     </inertial>
-    <collision name='collision'>
-      <origin xyz="0 0 0" rpy=" 0 0 0"/>
+    <collision name='right_collision'>
+      <origin xyz="0 0 0" rpy=" 0 1.5707 1.5707"/>
       <geometry>
          <cylinder length="0.05" radius="0.1"/>

Commit message: feat: Added command_robot callback function

File: my_robot/urdf/my_robot.xacro (robot description, xacro)
@@ -52,5 +52,5 @@
       />
     </inertial>
-    <collision name='left_collision'>
+    <collision name='collision'>
       <origin xyz="0 0 0" rpy=" 0 1.5707 1.5707"/>
       <geometry>
@@ -75,6 +75,6 @@
       />
     </inertial>
-    <collision name='right_collision'>
-      <origin xyz="0 0 0" rpy=" 0 1.5707 1.5707"/>
+    <collision name='collision'>
+      <origin xyz="0 0 0" rpy="0 1.5707 1.5707"/>
       <geometry>
          <cylinder length="0.05" radius="0.1"/>

Commit message: fix: Remove old model in world file

File: my_robot/urdf/my_robot.xacro (robot description, xacro)
@@ -34,4 +34,28 @@
       </geometry>
       <material name="blue"/>
+    </visual>
+    <collision name='back_caster_collision'>
+      <origin xyz="-0.15 0 -0.05" rpy=" 0 0 0"/>
+      <geometry>
+        <sphere radius="0.0499"/>
+      </geometry>
+    </collision>
+    <visual name='back_caster_visual'>
+      <origin xyz="-0.15 0 -0.05" rpy=" 0 0 0"/>
+      <geometry>
+        <sphere radius="0.05"/>
+      </geometry>
+    </visual>
+    <collision name='front_caster_collision'>
+      <origin xyz="0.15 0 -0.05" rpy=" 0 0 0"/>
+      <geometry>
+        <sphere radius="0.0499"/>
+      </geometry>
+    </collision>
+    <visual name='front_caster_visual'>
+      <origin xyz="0.15 0 -0.05" rpy=" 0 0 0"/>
+      <geometry>
+        <sphere radius="0.05"/>
+      </geometry>
     </visual>
   </link>
@@ -146,5 +170,5 @@
     <child link="right_wheel"/>
     <parent link="chassis"/>
-    <axis xyz="0 -1 0" rpy="0 0 0"/>
+    <axis xyz="0 1 0" rpy="0 0 0"/>
     <limit effort="10000" velocity="1000"/>
     <dynamics damping="1.0" friction="1.0"/>

Commit message: feat: Created 4 wheel robot with skid steer control

File: my_robot/urdf/my_robot.xacro (robot description, xacro)
@@ -2,7 +2,4 @@
 <robot name="my_robot" xmlns:xacro="http://www.ros.org/wiki/xacro">
  <xacro:include filename="$(find my_robot)/urdf/my_robot.gazebo" />
- <material name="blue">
-   <color rgba="0 0 0.8 1"/>
- </material>
  <link name="robot_footprint"></link>
   <joint name="robot_footprint_joint" type="fixed">
@@ -12,7 +9,7 @@
   </joint>
   <link name='chassis'>
-    <pose>0 0 0.1 0 0 0</pose>
-    <inertial>
-      <mass value="15.0"/>
+    <pose>0 0 0.2 0 0 0</pose>
+    <inertial>
+      <mass value="10.0"/>
       <origin xyz="0.0 0 0" rpy=" 0 0 0"/>
       <inertia
@@ -25,5 +22,5 @@
       <origin xyz="0 0 0" rpy=" 0 0 0"/>
       <geometry>
-        <box size=".4 .2 .1"/>
+        <box size=".25 .2 .2"/>
       </geometry>
     </collision>
@@ -31,76 +28,97 @@
       <origin xyz="0 0 0" rpy=" 0 0 0"/>
       <geometry>
-        <box size=".4 .2 .1"/>
-      </geometry>
-      <material name="blue"/>
-    </visual>
-    <collision name='back_caster_collision'>
-      <origin xyz="-0.15 0 -0.05" rpy=" 0 0 0"/>
-      <geometry>
-        <sphere radius="0.0499"/>
-      </geometry>
-    </collision>
-    <visual name='back_caster_visual'>
-      <origin xyz="-0.15 0 -0.05" rpy=" 0 0 0"/>
-      <geometry>
-        <sphere radius="0.05"/>
-      </geometry>
-    </visual>
-    <collision name='front_caster_collision'>
-      <origin xyz="0.15 0 -0.05" rpy=" 0 0 0"/>
-      <geometry>
-        <sphere radius="0.0499"/>
-      </geometry>
-    </collision>
-    <visual name='front_caster_visual'>
-      <origin xyz="0.15 0 -0.05" rpy=" 0 0 0"/>
-      <geometry>
-        <sphere radius="0.05"/>
-      </geometry>
-    </visual>
-  </link>
-  <link name='left_wheel'>
-     <visual>
-      <origin xyz="0.0 0 0" rpy=" 0 1.5707 1.5707"/>
-      <geometry>
-        <cylinder length="0.05" radius="0.1"/>
-      </geometry>
-    </visual>
-    <inertial>
-      <mass value="5.0"/>
-      <origin xyz="0.0 0 0" rpy=" 0 1.5707 1.5707"/>
-      <inertia
-          ixx="0.1" ixy="0" ixz="0"
-          iyy="0.1" iyz="0"
-          izz="0.1"
-      />
-    </inertial>
-    <collision name='collision'>
+        <box size=".25 .2 .2"/>
+      </geometry>
+    </visual>
+  </link>
+  <link name='front_left_wheel'>
+     <visual>
+      <origin xyz="0.0 0 0" rpy=" 0 1.5707 1.5707"/>
+      <geometry>
+        <cylinder length="0.04" radius="0.05"/>
+      </geometry>
+    </visual>
+    <inertial>
+      <mass value="5.0"/>
+      <origin xyz="0.0 0 0" rpy=" 0 1.5707 1.5707"/>
+      <inertia
+          ixx="0.1" ixy="0" ixz="0"
+          iyy="0.1" iyz="0"
+          izz="0.1"
+      />
+    </inertial>
+    <collision name='front_left_collision'>
       <origin xyz="0 0 0" rpy=" 0 1.5707 1.5707"/>
       <geometry>
-         <cylinder length="0.05" radius="0.1"/>
-      </geometry>
-    </collision>
-  </link>
-  <link name='right_wheel'>
-     <visual>
-      <origin xyz="0.0 0 0" rpy=" 0 1.5707 1.5707"/>
-      <geometry>
-        <cylinder length="0.05" radius="0.1"/>
-      </geometry>
-    </visual>
-    <inertial>
-      <mass value="5.0"/>
-      <origin xyz="0.0 0 0" rpy=" 0 1.5707 1.5707"/>
-      <inertia
-          ixx="0.1" ixy="0" ixz="0"
-          iyy="0.1" iyz="0"
-          izz="0.1"
-      />
-    </inertial>
-    <collision name='collision'>
+         <cylinder length="0.04" radius="0.05"/>
+      </geometry>
+    </collision>
+  </link>
+  <link name='front_right_wheel'>
+     <visual>
+      <origin xyz="0.0 0 0" rpy=" 0 1.5707 1.5707"/>
+      <geometry>
+        <cylinder length="0.04" radius="0.05"/>
+      </geometry>
+    </visual>
+    <inertial>
+      <mass value="5.0"/>
+      <origin xyz="0.0 0 0" rpy=" 0 1.5707 1.5707"/>
+      <inertia
+          ixx="0.1" ixy="0" ixz="0"
+          iyy="0.1" iyz="0"
+          izz="0.1"
+      />
+    </inertial>
+    <collision name='front_right_collision'>
       <origin xyz="0 0 0" rpy="0 1.5707 1.5707"/>
       <geometry>
-         <cylinder length="0.05" radius="0.1"/>
+         <cylinder length="0.04" radius="0.05"/>
+      </geometry>
+    </collision>
+  </link>
+<link name='rear_left_wheel'>
+     <visual>
+      <origin xyz="0.0 0 0" rpy=" 0 1.5707 1.5707"/>
+      <geometry>
+        <cylinder length="0.04" radius="0.05"/>
+      </geometry>
+    </visual>
+    <inertial>
+      <mass value="5.0"/>
+      <origin xyz="0.0 0 0" rpy=" 0 1.5707 1.5707"/>
+      <inertia
+          ixx="0.1" ixy="0" ixz="0"
+          iyy="0.1" iyz="0"
+          izz="0.1"
+      />
+    </inertial>
+    <collision name='rear_left_collision'>
+      <origin xyz="0 0 0" rpy=" 0 1.5707 1.5707"/>
+      <geometry>
+         <cylinder length="0.04" radius="0.05"/>
+      </geometry>
+    </collision>
+  </link>
+  <link name='rear_right_wheel'>
+     <visual>
+      <origin xyz="0.0 0 0" rpy=" 0 1.5707 1.5707"/>
+      <geometry>
+        <cylinder length="0.04" radius="0.05"/>
+      </geometry>
+    </visual>
+    <inertial>
+      <mass value="5.0"/>
+      <origin xyz="0.0 0 0" rpy=" 0 1.5707 1.5707"/>
+      <inertia
+          ixx="0.1" ixy="0" ixz="0"
+          iyy="0.1" iyz="0"
+          izz="0.1"
+      />
+    </inertial>
+    <collision name='rear_right_collision'>
+      <origin xyz="0 0 0" rpy="0 1.5707 1.5707"/>
+      <geometry>
+         <cylinder length="0.04" radius="0.05"/>
       </geometry>
     </collision>
@@ -151,5 +169,5 @@
       />
     </inertial>
-    <collision name='collision'>
+    <collision name='lidar_collision'>
       <origin xyz="0 0 0" rpy=" 0 0 0"/>
       <geometry>
@@ -158,15 +176,31 @@
     </collision>
   </link>
-  <joint type="continuous" name="left_wheel_hinge">
-    <origin xyz="0 0.15 0" rpy="0 0 0"/>
-    <child link="left_wheel"/>
-    <parent link="chassis"/>
-    <axis xyz="0 1 0" rpy="0 0 0"/>
-    <limit effort="10000" velocity="1000"/>
-    <dynamics damping="1.0" friction="1.0"/>
-  </joint>
-  <joint type="continuous" name="right_wheel_hinge">
-    <origin xyz="0 -0.15 0" rpy="0 0 0"/>
-    <child link="right_wheel"/>
+  <joint type="continuous" name="front_left_wheel_hinge">
+    <origin xyz="0.1 0.1 -0.1" rpy="0 0 0"/>
+    <child link="front_left_wheel"/>
+    <parent link="chassis"/>
+    <axis xyz="0 1 0" rpy="0 0 0"/>
+    <limit effort="10000" velocity="1000"/>
+    <dynamics damping="1.0" friction="1.0"/>
+  </joint>
+  <joint type="continuous" name="front_right_wheel_hinge">
+    <origin xyz="0.1 -0.1 -0.1" rpy="0 0 0"/>
+    <child link="front_right_wheel"/>
+    <parent link="chassis"/>
+    <axis xyz="0 1 0" rpy="0 0 0"/>
+    <limit effort="10000" velocity="1000"/>
+    <dynamics damping="1.0" friction="1.0"/>
+  </joint>
+  <joint type="continuous" name="rear_left_wheel_hinge">
+    <origin xyz="-0.1 0.1 -0.1" rpy="0 0 0"/>
+    <child link="rear_left_wheel"/>
+    <parent link="chassis"/>
+    <axis xyz="0 1 0" rpy="0 0 0"/>
+    <limit effort="10000" velocity="1000"/>
+    <dynamics damping="1.0" friction="1.0"/>
+  </joint>
+  <joint type="continuous" name="rear_right_wheel_hinge">
+    <origin xyz="-0.1 -0.1 -0.1" rpy="0 0 0"/>
+    <child link="rear_right_wheel"/>
     <parent link="chassis"/>
     <axis xyz="0 1 0" rpy="0 0 0"/>
@@ -175,5 +209,5 @@
   </joint>
   <joint type="fixed" name="camera_joint">
-    <origin xyz="0.2 0 0" rpy="0 0 0"/>
+    <origin xyz="0.1 0 0" rpy="0 0 0"/>
     <child link="camera"/>
     <parent link="chassis"/>

Commit message: fix: Improvements to robot design from feedback: * Include Odometry Topic, Odometry Frame * Enable BroadcastTF * Move camera location from being blocked * Remove delay in drive_bot.cpp * Move wheels to give more stability

File: my_robot/urdf/my_robot.xacro (robot description, xacro)
@@ -11,5 +11,5 @@
     <pose>0 0 0.2 0 0 0</pose>
     <inertial>
-      <mass value="10.0"/>
+      <mass value="12.0"/>
       <origin xyz="0.0 0 0" rpy=" 0 0 0"/>
       <inertia
@@ -29,4 +29,28 @@
       <geometry>
         <box size=".25 .2 .2"/>
+      </geometry>
+    </visual>
+    <collision name='front_caster_collision'>
+      <origin xyz="0.08 0 -0.1" rpy=" 0 0 0"/>
+      <geometry>
+        <sphere radius="0.0399"/>
+      </geometry>
+    </collision>
+    <visual name='front_caster_visual'>
+      <origin xyz="0.08 0 -0.1" rpy=" 0 0 0"/>
+      <geometry>
+        <sphere radius="0.04"/>
+      </geometry>
+    </visual>
+    <collision name='rear_caster_collision'>
+      <origin xyz="-0.08 0 -0.1" rpy=" 0 0 0"/>
+      <geometry>
+        <sphere radius="0.0399"/>
+      </geometry>
+    </collision>
+    <visual name='rear_caster_visual'>
+      <origin xyz="-0.08 0 -0.1" rpy=" 0 0 0"/>
+      <geometry>
+        <sphere radius="0.04"/>
       </geometry>
     </visual>
@@ -126,5 +150,5 @@
   <link name='camera'>
      <visual>
-      <origin xyz="0.0 0 0" rpy=" 0 0 0"/>
+      <origin xyz="0.025 0 0" rpy=" 0 0 0"/>
       <geometry>
         <box size=".05 .05 .05"/>
@@ -136,5 +160,5 @@
         <box size=".05 .05 .05"/>
       </geometry>
-      <origin xyz="0.0 0 0" rpy=" 0 0 0"/>
+      <origin xyz="0 0 0" rpy=" 0 0 0"/>
       <inertia
 	ixx="1e-6" ixy="0" ixz="0"
@@ -152,5 +176,5 @@
   <link name='hokuyo'>
      <visual>
-      <origin xyz="0.0 0 0" rpy=" 0 0 0"/>
+      <origin xyz="0 0 0" rpy=" 0 0 0"/>
       <geometry>
 	<mesh filename= "package://my_robot/meshes/hokuyo.dae"/>
@@ -160,7 +184,7 @@
       <mass value="1e-5"/>
       <geometry>
-        <box size=".05 .05 .05"/>
-      </geometry>
-      <origin xyz="0.0 0 0" rpy=" 0 0 0"/>
+        <box size=".04 .04 .04"/>
+      </geometry>
+      <origin xyz="0 0 0" rpy=" 0 0 0"/>
       <inertia
 	ixx="1e-6" ixy="0" ixz="0"
@@ -177,5 +201,5 @@
   </link>
   <joint type="continuous" name="front_left_wheel_hinge">
-    <origin xyz="0.1 0.1 -0.1" rpy="0 0 0"/>
+    <origin xyz="0.1 0.12 -0.1" rpy="0 0 0"/>
     <child link="front_left_wheel"/>
     <parent link="chassis"/>
@@ -185,5 +209,5 @@
   </joint>
   <joint type="continuous" name="front_right_wheel_hinge">
-    <origin xyz="0.1 -0.1 -0.1" rpy="0 0 0"/>
+    <origin xyz="0.1 -0.12 -0.1" rpy="0 0 0"/>
     <child link="front_right_wheel"/>
     <parent link="chassis"/>
@@ -193,5 +217,5 @@
   </joint>
   <joint type="continuous" name="rear_left_wheel_hinge">
-    <origin xyz="-0.1 0.1 -0.1" rpy="0 0 0"/>
+    <origin xyz="-0.1 0.12 -0.1" rpy="0 0 0"/>
     <child link="rear_left_wheel"/>
     <parent link="chassis"/>
@@ -201,5 +225,5 @@
   </joint>
   <joint type="continuous" name="rear_right_wheel_hinge">
-    <origin xyz="-0.1 -0.1 -0.1" rpy="0 0 0"/>
+    <origin xyz="-0.1 -0.12 -0.1" rpy="0 0 0"/>
     <child link="rear_right_wheel"/>
     <parent link="chassis"/>
@@ -209,5 +233,5 @@
   </joint>
   <joint type="fixed" name="camera_joint">
-    <origin xyz="0.1 0 0" rpy="0 0 0"/>
+    <origin xyz="0.1 0 0.125" rpy="0 0 0"/>
     <child link="camera"/>
     <parent link="chassis"/>
@@ -217,5 +241,5 @@
   </joint>
   <joint type="fixed" name="hokuyo_joint">
-    <origin xyz="0.15 0 0.1" rpy="0 0 0"/>
+    <origin xyz="-0.1 0.05 0.125" rpy="0 0 0"/>
     <child link="hokuyo"/>
     <parent link="chassis"/>

Commit message: feat:Add generated map for localisation

File: my_robot/urdf/my_robot.xacro (robot description, xacro)
@@ -203,5 +203,5 @@
     <origin xyz="0.1 0.12 -0.1" rpy="0 0 0"/>
     <child link="front_left_wheel"/>
-    <parent link="chassis"/>
+    <parent link="robot_footprint"/>
     <axis xyz="0 1 0" rpy="0 0 0"/>
     <limit effort="10000" velocity="1000"/>

Commit message: fix: Change left wheel back to child of chassis  (had no effect)

File: my_robot/urdf/my_robot.xacro (robot description, xacro)
@@ -203,5 +203,5 @@
     <origin xyz="0.1 0.12 -0.1" rpy="0 0 0"/>
     <child link="front_left_wheel"/>
-    <parent link="robot_footprint"/>
+    <parent link="chassis"/>
     <axis xyz="0 1 0" rpy="0 0 0"/>
     <limit effort="10000" velocity="1000"/>

Commit message: feat: Increase map size, move robot origin, tweak ACML parameters

File: my_robot/urdf/my_robot.xacro (robot description, xacro)
@@ -9,8 +9,8 @@
   </joint>
   <link name='chassis'>
-    <pose>0 0 0.2 0 0 0</pose>
+    <pose>0 0 0 0 0 0</pose>
     <inertial>
       <mass value="12.0"/>
-      <origin xyz="0.0 0 0" rpy=" 0 0 0"/>
+      <origin xyz="0.0 0 0.2" rpy=" 0 0 0"/>
       <inertia
           ixx="0.1" ixy="0" ixz="0"

Commit message: fix: Tweak amcl values, add rviz config file

File: my_robot/urdf/my_robot.xacro (robot description, xacro)
@@ -9,8 +9,8 @@
   </joint>
   <link name='chassis'>
-    <pose>0 0 0 0 0 0</pose>
+    <pose>0 0 -0.4 0 0 0</pose>
     <inertial>
       <mass value="12.0"/>
-      <origin xyz="0.0 0 0.2" rpy=" 0 0 0"/>
+      <origin xyz="0.0 0 0" rpy=" 0 0 0"/>
       <inertia
           ixx="0.1" ixy="0" ixz="0"
@@ -28,29 +28,5 @@
       <origin xyz="0 0 0" rpy=" 0 0 0"/>
       <geometry>
-        <box size=".25 .2 .2"/>
-      </geometry>
-    </visual>
-    <collision name='front_caster_collision'>
-      <origin xyz="0.08 0 -0.1" rpy=" 0 0 0"/>
-      <geometry>
-        <sphere radius="0.0399"/>
-      </geometry>
-    </collision>
-    <visual name='front_caster_visual'>
-      <origin xyz="0.08 0 -0.1" rpy=" 0 0 0"/>
-      <geometry>
-        <sphere radius="0.04"/>
-      </geometry>
-    </visual>
-    <collision name='rear_caster_collision'>
-      <origin xyz="-0.08 0 -0.1" rpy=" 0 0 0"/>
-      <geometry>
-        <sphere radius="0.0399"/>
-      </geometry>
-    </collision>
-    <visual name='rear_caster_visual'>
-      <origin xyz="-0.08 0 -0.1" rpy=" 0 0 0"/>
-      <geometry>
-        <sphere radius="0.04"/>
+        <box size=".25 .2 .1"/>
       </geometry>
     </visual>
@@ -201,5 +177,5 @@
   </link>
   <joint type="continuous" name="front_left_wheel_hinge">
-    <origin xyz="0.1 0.12 -0.1" rpy="0 0 0"/>
+    <origin xyz="0.1 0.11 -0.05" rpy="0 0 0"/>
     <child link="front_left_wheel"/>
     <parent link="chassis"/>
@@ -209,5 +185,5 @@
   </joint>
   <joint type="continuous" name="front_right_wheel_hinge">
-    <origin xyz="0.1 -0.12 -0.1" rpy="0 0 0"/>
+    <origin xyz="0.1 -0.11 -0.05" rpy="0 0 0"/>
     <child link="front_right_wheel"/>
     <parent link="chassis"/>
@@ -217,5 +193,5 @@
   </joint>
   <joint type="continuous" name="rear_left_wheel_hinge">
-    <origin xyz="-0.1 0.12 -0.1" rpy="0 0 0"/>
+    <origin xyz="-0.1 0.11 -0.050" rpy="0 0 0"/>
     <child link="rear_left_wheel"/>
     <parent link="chassis"/>
@@ -225,5 +201,5 @@
   </joint>
   <joint type="continuous" name="rear_right_wheel_hinge">
-    <origin xyz="-0.1 -0.12 -0.1" rpy="0 0 0"/>
+    <origin xyz="-0.1 -0.11 -0.05" rpy="0 0 0"/>
     <child link="rear_right_wheel"/>
     <parent link="chassis"/>
@@ -233,5 +209,5 @@
   </joint>
   <joint type="fixed" name="camera_joint">
-    <origin xyz="0.1 0 0.125" rpy="0 0 0"/>
+    <origin xyz="0.05 0 0.05" rpy="0 0 0"/>
     <child link="camera"/>
     <parent link="chassis"/>
@@ -241,5 +217,5 @@
   </joint>
   <joint type="fixed" name="hokuyo_joint">
-    <origin xyz="-0.1 0.05 0.125" rpy="0 0 0"/>
+    <origin xyz="-0.1 0.05 0.05" rpy="0 0 0"/>
     <child link="hokuyo"/>
     <parent link="chassis"/>

Commit message: fix: Correct topic name in costmap parameters, move laser to fron to robot

File: my_robot/urdf/my_robot.xacro (robot description, xacro)
@@ -209,13 +209,13 @@
   </joint>
   <joint type="fixed" name="camera_joint">
+    <origin xyz="-0.1 0.05 0.05" rpy="0 0 0"/>
+    <child link="camera"/>
+    <parent link="chassis"/>
+    <axis xyz="0 1 0" rpy="0 0 0"/>
+    <limit effort="10000" velocity="1000"/>
+    <dynamics damping="1.0" friction="1.0"/>
+  </joint>
+  <joint type="fixed" name="hokuyo_joint">
     <origin xyz="0.05 0 0.05" rpy="0 0 0"/>
-    <child link="camera"/>
-    <parent link="chassis"/>
-    <axis xyz="0 1 0" rpy="0 0 0"/>
-    <limit effort="10000" velocity="1000"/>
-    <dynamics damping="1.0" friction="1.0"/>
-  </joint>
-  <joint type="fixed" name="hokuyo_joint">
-    <origin xyz="-0.1 0.05 0.05" rpy="0 0 0"/>
     <child link="hokuyo"/>
     <parent link="chassis"/>
